File: OverdrivePedal_RevB/OverdrivePedal_RevB.sch (KiCad schematic (older format))
At the start: 14 parts, among them J1 Conn_01x02, J2 Conn_01x02, J3 Conn_01x03, J4 Conn_01x03, J5 Conn_01x03, J6 Conn_01x02, U1 TL072

Commit message: modified RevB
Parts:
- removed U1: TL072, Package_SO:TSSOP-8_4.4x3mm_P0.65mm, symbol Amplifier_Operational:TL072
- added U2: TL071, Package_SO:SOIC-8_3.9x4.9mm_P1.27mm, symbol Amplifier_Operational:TL071
Connections:
- wire segments 63 -> 53
- no-connect marks 0 -> 2
Other:
- moved on the sheet: C2, C7, C9
Changed lines of the file:
@@
 $EndComp
 Wire Wire Line
-	5700 2950 5400 2950
-Wire Wire Line
-	5400 2950 5400 3600
+	5700 2850 5400 2850
+Wire Wire Line
+	5400 2850 5400 3600
 Wire Wire Line
 	5400 3600 5900 3600
@@
 	6100 3600 6750 3600
 Wire Wire Line
-	6750 3600 6750 2850
-Wire Wire Line
-	6750 2850 6300 2850
+	6750 3600 6750 2750
+Wire Wire Line
+	6750 2750 6300 2750
 Wire Wire Line
 	6000 3800 6000 3600
@@
 	1    0    0    -1
 $EndComp
-Connection ~ 6750 2850
+Connection ~ 6750 2750
 $Comp
 L Device:R R3
@@
 $EndComp
 Wire Wire Line
-	8050 3450 8050 2850
+	8050 3450 8050 2750
 Wire Wire Line
 	8050 3750 8050 4450
@@
 	4700 6450 4700 6650
 Wire Wire Line
-	2450 6150 1450 6150
+	2450 6150 1700 6150
 $Comp
 L Connector_Generic:Conn_01x02 J2
 U 1 1 5E669F6B
-P 1250 6150
-F 0 "J2" H 1168 6367 50  0000 C CNN
-F 1 "Conn_01x02" H 1168 6276 50  0000 C CNN
-F 2 "Connector_PinHeader_2.54mm:PinHeader_1x02_P2.54mm_Vertical" H 1250 6150 50  0001 C CNN
-F 3 "~" H 1250 6150 50  0001 C CNN
-	1    1250 6150
+P 1500 6150
+F 0 "J2" H 1418 6367 50  0000 C CNN
+F 1 "Conn_01x02" H 1418 6276 50  0000 C CNN
+F 2 "Connector_PinHeader_2.54mm:PinHeader_1x02_P2.54mm_Vertical" H 1500 6150 50  0001 C CNN
+F 3 "~" H 1500 6150 50  0001 C CNN
+	1    1500 6150
 	-1   0    0    -1
 $EndComp
 Wire Wire Line
-	1450 6250 1850 6250
-Wire Wire Line
-	1850 6250 1850 6750
+	1700 6250 2100 6250
+Wire Wire Line
+	2100 6250 2100 6750
 $Comp
 L power:GNDS #PWR02
 U 1 1 5E66AC31
-P 1850 6750
-F 0 "#PWR02" H 1850 6500 50  0001 C CNN
-F 1 "GNDS" H 1855 6577 50  0000 C CNN
-F 2 "" H 1850 6750 50  0001 C CNN
-F 3 "" H 1850 6750 50  0001 C CNN
-	1    1850 6750
+P 2100 6750
+F 0 "#PWR02" H 2100 6500 50  0001 C CNN
+F 1 "GNDS" H 2105 6577 50  0000 C CNN
+F 2 "" H 2100 6750 50  0001 C CNN
+F 3 "" H 2100 6750 50  0001 C CNN
+	1    2100 6750
 	1    0    0    -1
 $EndComp
@@
 Wire Wire Line
 	3800 3350 3800 2650
-Wire Wire Line
-	3800 2650 4300 2650
 Wire Wire Line
 	3800 3650 3800 4550
@@
 Wire Wire Line
 	1700 2050 3000 2050
-Connection ~ 3800 2650
 Wire Wire Line
 	9600 2150 9500 2150
@@
 	8850 2150 9100 2150
 Wire Wire Line
-	9100 2150 9100 2850
-Connection ~ 8050 2850
-Wire Wire Line
-	8050 2850 9100 2850
+	9100 2150 9100 2750
+Connection ~ 8050 2750
+Wire Wire Line
+	8050 2750 9100 2750
 Text Notes 9650 1900 0    50   ~ 0
 Output Jack
@@
 Input Jack
 $Comp
-L Amplifier_Operational:TL072 U1
-U 1 1 5E645B4B
-P 4600 2750
-F 0 "U1" H 4600 3117 50  0000 C CNN
-F 1 "TL072" H 4600 3026 50  0000 C CNN
-F 2 "Package_SO:TSSOP-8_4.4x3mm_P0.65mm" H 4600 2750 50  0001 C CNN
-F 3 "http://www.ti.com/lit/ds/symlink/tl071.pdf" H 4600 2750 50  0001 C CNN
-	1    4600 2750
-	1    0    0    -1
-$EndComp
-$Comp
-L Amplifier_Operational:TL072 U1
-U 2 1 5E646D18
-P 6000 2850
-F 0 "U1" H 6000 3217 50  0000 C CNN
-F 1 "TL072" H 6000 3126 50  0000 C CNN
-F 2 "Package_SO:TSSOP-8_4.4x3mm_P0.65mm" H 6000 2850 50  0001 C CNN
-F 3 "http://www.ti.com/lit/ds/symlink/tl071.pdf" H 6000 2850 50  0001 C CNN
-	2    6000 2850
-	1    0    0    -1
-$EndComp
-$Comp
-L Amplifier_Operational:TL072 U1
-U 3 1 5E64953A
-P 6000 6300
-F 0 "U1" H 5958 6346 50  0000 L CNN
-F 1 "TL072" H 5958 6255 50  0000 L CNN
-F 2 "Package_SO:TSSOP-8_4.4x3mm_P0.65mm" H 6000 6300 50  0001 C CNN
-F 3 "http://www.ti.com/lit/ds/symlink/tl071.pdf" H 6000 6300 50  0001 C CNN
-	3    6000 6300
-	1    0    0    -1
-$EndComp
-Wire Wire Line
-	5900 6000 5900 5900
-$Comp
 L power:+5V #PWR07
 U 1 1 5E654320
-P 5900 5500
-F 0 "#PWR07" H 5900 5350 50  0001 C CNN
-F 1 "+5V" H 5915 5673 50  0000 C CNN
-F 2 "" H 5900 5500 50  0001 C CNN
-F 3 "" H 5900 5500 50  0001 C CNN
-	1    5900 5500
+P 5650 5975
+F 0 "#PWR07" H 5650 5825 50  0001 C CNN
+F 1 "+5V" H 5665 6148 50  0000 C CNN
+F 2 "" H 5650 5975 50  0001 C CNN
+F 3 "" H 5650 5975 50  0001 C CNN
+	1    5650 5975
 	1    0    0    -1
 $EndComp
@@
 L power:-5V #PWR08
 U 1 1 5E65531A
-P 5900 7050
-F 0 "#PWR08" H 5900 7150 50  0001 C CNN
-F 1 "-5V" H 5915 7223 50  0000 C CNN
-F 2 "" H 5900 7050 50  0001 C CNN
-F 3 "" H 5900 7050 50  0001 C CNN
-	1    5900 7050
-	-1   0    0    1
-$EndComp
-Wire Wire Line
-	5900 6600 5900 6650
-Wire Wire Line
-	4900 2750 5050 2750
-Wire Wire Line
-	4300 2850 4150 2850
-Wire Wire Line
-	4150 2850 4150 3150
-Wire Wire Line
-	4150 3150 5050 3150
-Wire Wire Line
-	5050 3150 5050 2750
-Connection ~ 5050 2750
-Wire Wire Line
-	5050 2750 5700 2750
+P 6250 5975
+F 0 "#PWR08" H 6250 6075 50  0001 C CNN
+F 1 "-5V" H 6265 6148 50  0000 C CNN
+F 2 "" H 6250 5975 50  0001 C CNN
+F 3 "" H 6250 5975 50  0001 C CNN
+	1    6250 5975
+	1    0    0    -1
+$EndComp
 Wire Wire Line
 	2750 2650 3100 2650
 Wire Wire Line
-	6750 2850 7250 2850
+	6750 2750 7250 2750
 $Comp
 L Device:C C2
 U 1 1 5E68E4E0
-P 7400 2850
-F 0 "C2" V 7148 2850 50  0000 C CNN
-F 1 "1uF" V 7239 2850 50  0000 C CNN
-F 2 "Capacitor_SMD:C_0805_2012Metric_Pad1.15x1.40mm_HandSolder" H 7438 2700 50  0001 C CNN
-F 3 "~" H 7400 2850 50  0001 C CNN
-	1    7400 2850
+P 7400 2750
+F 0 "C2" V 7148 2750 50  0000 C CNN
+F 1 "1uF" V 7239 2750 50  0000 C CNN
+F 2 "Capacitor_SMD:C_0805_2012Metric_Pad1.15x1.40mm_HandSolder" H 7438 2600 50  0001 C CNN
+F 3 "~" H 7400 2750 50  0001 C CNN
+	1    7400 2750
 	0    1    1    0
 $EndComp
 Wire Wire Line
-	7550 2850 8050 2850
+	7550 2750 8050 2750
 $Comp
 L Device:C C1
@@
 L Device:C C?
 U 1 1 5E6944EB
-P 6500 6850
+P 6250 6275
 AR Path="/5E6165F4/5E6944EB" Ref="C?"  Part="1"
 AR Path="/5E6A8284/5E6944EB" Ref="C?"  Part="1"
 AR Path="/5E6944EB" Ref="C9"  Part="1"
-F 0 "C9" H 6615 6896 50  0000 L CNN
-F 1 "100nF" H 6615 6805 50  0000 L CNN
-F 2 "Capacitor_SMD:C_0805_2012Metric_Pad1.15x1.40mm_HandSolder" H 6538 6700 50  0001 C CNN
-F 3 "~" H 6500 6850 50  0001 C CNN
-	1    6500 6850
-	1    0    0    -1
-$EndComp
-Wire Wire Line
-	6500 6700 6500 6650
-Wire Wire Line
-	6500 7000 6500 7050
+F 0 "C9" H 6365 6321 50  0000 L CNN
+F 1 "100nF" H 6365 6230 50  0000 L CNN
+F 2 "Capacitor_SMD:C_0805_2012Metric_Pad1.15x1.40mm_HandSolder" H 6288 6125 50  0001 C CNN
+F 3 "~" H 6250 6275 50  0001 C CNN
+	1    6250 6275
+	1    0    0    -1
+$EndComp
+Wire Wire Line
+	6250 6425 6250 6550
 $Comp
 L power:GNDS #PWR?
 U 1 1 5E6944F3
-P 6500 7050
+P 6250 6550
 AR Path="/5E6165F4/5E6944F3" Ref="#PWR?"  Part="1"
 AR Path="/5E6944F3" Ref="#PWR0101"  Part="1"
-F 0 "#PWR0101" H 6500 6800 50  0001 C CNN
-F 1 "GNDS" H 6505 6877 50  0000 C CNN
-F 2 "" H 6500 7050 50  0001 C CNN
-F 3 "" H 6500 7050 50  0001 C CNN
-	1    6500 7050
-	1    0    0    -1
-$EndComp
-Wire Wire Line
-	6500 6650 5900 6650
-Connection ~ 5900 6650
-Wire Wire Line
-	5900 6650 5900 7050
+F 0 "#PWR0101" H 6250 6300 50  0001 C CNN
+F 1 "GNDS" H 6255 6377 50  0000 C CNN
+F 2 "" H 6250 6550 50  0001 C CNN
+F 3 "" H 6250 6550 50  0001 C CNN
+	1    6250 6550
+	1    0    0    -1
+$EndComp
 $Comp
 L Device:C C?
 U 1 1 5E6978C7
-P 6500 5700
+P 5650 6275
 AR Path="/5E6165F4/5E6978C7" Ref="C?"  Part="1"
 AR Path="/5E6A8284/5E6978C7" Ref="C?"  Part="1"
 AR Path="/5E6978C7" Ref="C7"  Part="1"
-F 0 "C7" H 6615 5746 50  0000 L CNN
-F 1 "100nF" H 6615 5655 50  0000 L CNN
-F 2 "Capacitor_SMD:C_0805_2012Metric_Pad1.15x1.40mm_HandSolder" H 6538 5550 50  0001 C CNN
-F 3 "~" H 6500 5700 50  0001 C CNN
-	1    6500 5700
-	1    0    0    1
-$EndComp
-Wire Wire Line
-	6500 5850 6500 5900
-Wire Wire Line
-	6500 5550 6500 5500
+F 0 "C7" H 5765 6321 50  0000 L CNN
+F 1 "100nF" H 5765 6230 50  0000 L CNN
+F 2 "Capacitor_SMD:C_0805_2012Metric_Pad1.15x1.40mm_HandSolder" H 5688 6125 50  0001 C CNN
+F 3 "~" H 5650 6275 50  0001 C CNN
+	1    5650 6275
+	-1   0    0    -1
+$EndComp
+Wire Wire Line
+	5650 6425 5650 6550
 $Comp
 L power:GNDS #PWR?
 U 1 1 5E6978CF
-P 6500 5500
+P 5650 6550
 AR Path="/5E6165F4/5E6978CF" Ref="#PWR?"  Part="1"
 AR Path="/5E6978CF" Ref="#PWR0102"  Part="1"
-F 0 "#PWR0102" H 6500 5250 50  0001 C CNN
-F 1 "GNDS" H 6505 5327 50  0000 C CNN
-F 2 "" H 6500 5500 50  0001 C CNN
-F 3 "" H 6500 5500 50  0001 C CNN
-	1    6500 5500
-	1    0    0    1
-$EndComp
-Wire Wire Line
-	6500 5900 5900 5900
-Connection ~ 5900 5900
-Wire Wire Line
-	5900 5900 5900 5500
+F 0 "#PWR0102" H 5650 6300 50  0001 C CNN
+F 1 "GNDS" H 5655 6377 50  0000 C CNN
+F 2 "" H 5650 6550 50  0001 C CNN
+F 3 "" H 5650 6550 50  0001 C CNN
+	1    5650 6550
+	-1   0    0    -1
+$EndComp
 $Comp
 L power:GNDS #PWR0103
@@
 Wire Wire Line
 	8050 4450 8050 4650
-Connection ~ 1550 1650
+$Comp
+L Amplifier_Operational:TL071 U2
+U 1 1 5E6CAB10
+P 6000 2750
+F 0 "U2" H 6350 3100 50  0000 L CNN
+F 1 "TL071" H 6350 3000 50  0000 L CNN
+F 2 "Package_SO:SOIC-8_3.9x4.9mm_P1.27mm" H 6050 2800 50  0001 C CNN
+F 3 "http://www.ti.com/lit/ds/symlink/tl071.pdf" H 6150 2900 50  0001 C CNN
+	1    6000 2750
+	1    0    0    -1
+$EndComp
+Wire Wire Line
+	3800 2650 5700 2650
+Connection ~ 3800 2650
+$Comp
+L power:+5V #PWR0104
+U 1 1 5E6E3613
+P 5900 2400
+F 0 "#PWR0104" H 5900 2250 50  0001 C CNN
+F 1 "+5V" H 5915 2573 50  0000 C CNN
+F 2 "" H 5900 2400 50  0001 C CNN
+F 3 "" H 5900 2400 50  0001 C CNN
+	1    5900 2400
+	1    0    0    -1
+$EndComp
+Wire Wire Line
+	5900 2450 5900 2400
+$Comp
+L power:-5V #PWR0105
+U 1 1 5E6E9715
+P 5900 3125
+F 0 "#PWR0105" H 5900 3225 50  0001 C CNN
+F 1 "-5V" H 5915 3298 50  0000 C CNN
+F 2 "" H 5900 3125 50  0001 C CNN
+F 3 "" H 5900 3125 50  0001 C CNN
+	1    5900 3125
+	-1   0    0    1
+$EndComp
+Wire Wire Line
+	5900 3050 5900 3125
+NoConn ~ 6000 3050
+NoConn ~ 6100 3050
+Wire Wire Line
+	5650 5975 5650 6125
+Wire Wire Line
+	6250 5975 6250 6125
 $EndSCHEMATC

Commit message: Added 2 x RGB LEDS
Parts:
- added D2, D3: LED_RGBA, LED_THT:LED_D5.0mm-4_RGB_Wide_Pins, symbol Device:LED_RGBA
- added R4, R5, R6, R7, R8, R9: R, Resistor_SMD:R_0805_2012Metric_Pad1.15x1.40mm_HandSolder, symbol Device:R
Connections:
- wire segments 53 -> 77
Changed lines of the file:
@@
 	8050 3450 8050 2750
 Wire Wire Line
-	8050 3750 8050 4450
+	8050 3750 8050 4000
 $Comp
 L power:GNDS #PWR09
 U 1 1 5E604332
-P 8050 4650
-F 0 "#PWR09" H 8050 4400 50  0001 C CNN
-F 1 "GNDS" H 8055 4477 50  0000 C CNN
-F 2 "" H 8050 4650 50  0001 C CNN
-F 3 "" H 8050 4650 50  0001 C CNN
-	1    8050 4650
+P 8050 4200
+F 0 "#PWR09" H 8050 3950 50  0001 C CNN
+F 1 "GNDS" H 8055 4027 50  0000 C CNN
+F 2 "" H 8050 4200 50  0001 C CNN
+F 3 "" H 8050 4200 50  0001 C CNN
+	1    8050 4200
 	1    0    0    -1
 $EndComp
@@
 	9600 2150 9500 2150
 Wire Wire Line
-	9500 2150 9500 4200
+	9500 2150 9500 3750
 $Comp
 L power:GNDS #PWR010
 U 1 1 5E6796F4
-P 9500 4200
-F 0 "#PWR010" H 9500 3950 50  0001 C CNN
-F 1 "GNDS" H 9505 4027 50  0000 C CNN
-F 2 "" H 9500 4200 50  0001 C CNN
-F 3 "" H 9500 4200 50  0001 C CNN
-	1    9500 4200
+P 9500 3750
+F 0 "#PWR010" H 9500 3500 50  0001 C CNN
+F 1 "GNDS" H 9505 3577 50  0000 C CNN
+F 2 "" H 9500 3750 50  0001 C CNN
+F 3 "" H 9500 3750 50  0001 C CNN
+	1    9500 3750
 	1    0    0    -1
 $EndComp
@@
 	2000 2150 2000 4000
 Wire Wire Line
-	8400 4450 8050 4450
-Wire Wire Line
-	8400 4650 8400 4450
+	8400 4000 8050 4000
+Wire Wire Line
+	8400 4200 8400 4000
 $Comp
 L power:PWR_FLAG #FLG0101
 U 1 1 5E6B8B4F
-P 8400 4650
-F 0 "#FLG0101" H 8400 4725 50  0001 C CNN
-F 1 "PWR_FLAG" H 8400 4823 50  0000 C CNN
-F 2 "" H 8400 4650 50  0001 C CNN
-F 3 "~" H 8400 4650 50  0001 C CNN
-	1    8400 4650
-	-1   0    0    1
-$EndComp
-Connection ~ 8050 4450
-Wire Wire Line
-	8050 4450 8050 4650
+P 8400 4200
+F 0 "#FLG0101" H 8400 4275 50  0001 C CNN
+F 1 "PWR_FLAG" H 8400 4373 50  0000 C CNN
+F 2 "" H 8400 4200 50  0001 C CNN
+F 3 "~" H 8400 4200 50  0001 C CNN
+	1    8400 4200
+	-1   0    0    1
+$EndComp
+Connection ~ 8050 4000
+Wire Wire Line
+	8050 4000 8050 4200
 $Comp
 L Amplifier_Operational:TL071 U2
@@
 Wire Wire Line
 	6250 5975 6250 6125
+$Comp
+L Device:LED_RGBA D3
+U 1 1 5E722548
+P 9900 5300
+F 0 "D3" V 9854 5660 50  0000 L CNN
+F 1 "LED_RGBA" V 9945 5660 50  0000 L CNN
+F 2 "LED_THT:LED_D5.0mm-4_RGB_Wide_Pins" H 9900 5250 50  0001 C CNN
+F 3 "~" H 9900 5250 50  0001 C CNN
+	1    9900 5300
+	0    -1   -1   0
+$EndComp
+$Comp
+L Device:LED_RGBA D2
+U 1 1 5E72451F
+P 8450 5300
+F 0 "D2" V 8404 5660 50  0000 L CNN
+F 1 "LED_RGBA" V 8495 5660 50  0000 L CNN
+F 2 "LED_THT:LED_D5.0mm-4_RGB_Wide_Pins" H 8450 5250 50  0001 C CNN
+F 3 "~" H 8450 5250 50  0001 C CNN
+	1    8450 5300
+	0    -1   -1   0
+$EndComp
+$Comp
+L Device:R R9
+U 1 1 5E7266E9
+P 10100 5750
+F 0 "R9" H 10170 5796 50  0000 L CNN
+F 1 "R" H 10170 5705 50  0000 L CNN
+F 2 "Resistor_SMD:R_0805_2012Metric_Pad1.15x1.40mm_HandSolder" V 10030 5750 50  0001 C CNN
+F 3 "~" H 10100 5750 50  0001 C CNN
+	1    10100 5750
+	-1   0    0    1
+$EndComp
+$Comp
+L Device:R R8
+U 1 1 5E726B3F
+P 9900 5750
+F 0 "R8" H 9970 5796 50  0000 L CNN
+F 1 "R" H 9970 5705 50  0000 L CNN
+F 2 "Resistor_SMD:R_0805_2012Metric_Pad1.15x1.40mm_HandSolder" V 9830 5750 50  0001 C CNN
+F 3 "~" H 9900 5750 50  0001 C CNN
+	1    9900 5750
+	-1   0    0    1
+$EndComp
+$Comp
+L Device:R R7
+U 1 1 5E727007
+P 9700 5750
+F 0 "R7" H 9770 5796 50  0000 L CNN
+F 1 "R" H 9770 5705 50  0000 L CNN
+F 2 "Resistor_SMD:R_0805_2012Metric_Pad1.15x1.40mm_HandSolder" V 9630 5750 50  0001 C CNN
+F 3 "~" H 9700 5750 50  0001 C CNN
+	1    9700 5750
+	-1   0    0    1
+$EndComp
+$Comp
+L Device:R R6
+U 1 1 5E727E16
+P 8650 5750
+F 0 "R6" H 8720 5796 50  0000 L CNN
+F 1 "R" H 8720 5705 50  0000 L CNN
+F 2 "Resistor_SMD:R_0805_2012Metric_Pad1.15x1.40mm_HandSolder" V 8580 5750 50  0001 C CNN
+F 3 "~" H 8650 5750 50  0001 C CNN
+	1    8650 5750
+	-1   0    0    1
+$EndComp
+$Comp
+L Device:R R5
+U 1 1 5E727E1C
+P 8450 5750
+F 0 "R5" H 8520 5796 50  0000 L CNN
+F 1 "R" H 8520 5705 50  0000 L CNN
+F 2 "Resistor_SMD:R_0805_2012Metric_Pad1.15x1.40mm_HandSolder" V 8380 5750 50  0001 C CNN
+F 3 "~" H 8450 5750 50  0001 C CNN
+	1    8450 5750
+	-1   0    0    1
+$EndComp
+$Comp
+L Device:R R4
+U 1 1 5E727E22
+P 8250 5750
+F 0 "R4" H 8320 5796 50  0000 L CNN
+F 1 "R" H 8320 5705 50  0000 L CNN
+F 2 "Resistor_SMD:R_0805_2012Metric_Pad1.15x1.40mm_HandSolder" V 8180 5750 50  0001 C CNN
+F 3 "~" H 8250 5750 50  0001 C CNN
+	1    8250 5750
+	-1   0    0    1
+$EndComp
+Wire Wire Line
+	10100 5600 10100 5500
+Wire Wire Line
+	9900 5600 9900 5500
+Wire Wire Line
+	9700 5600 9700 5500
+Wire Wire Line
+	8650 5600 8650 5500
+Wire Wire Line
+	8450 5600 8450 5500
+Wire Wire Line
+	8250 5600 8250 5500
+Wire Wire Line
+	9900 5100 9900 4950
+Wire Wire Line
+	8450 5100 8450 4950
+$Comp
+L power:GNDS #PWR0108
+U 1 1 5E73B1FE
+P 9150 6150
+F 0 "#PWR0108" H 9150 5900 50  0001 C CNN
+F 1 "GNDS" H 9155 5977 50  0000 C CNN
+F 2 "" H 9150 6150 50  0001 C CNN
+F 3 "" H 9150 6150 50  0001 C CNN
+	1    9150 6150
+	1    0    0    -1
+$EndComp
+$Comp
+L power:+5V #PWR0109
+U 1 1 5E73B611
+P 9150 4850
+F 0 "#PWR0109" H 9150 4700 50  0001 C CNN
+F 1 "+5V" H 9165 5023 50  0000 C CNN
+F 2 "" H 9150 4850 50  0001 C CNN
+F 3 "" H 9150 4850 50  0001 C CNN
+	1    9150 4850
+	1    0    0    -1
+$EndComp
+Wire Wire Line
+	9150 6150 9150 6050
+Wire Wire Line
+	9150 6050 9700 6050
+Wire Wire Line
+	10100 6050 10100 5900
+Wire Wire Line
+	9900 6050 9900 5900
+Connection ~ 9900 6050
+Wire Wire Line
+	9900 6050 10100 6050
+Wire Wire Line
+	9700 6050 9700 5900
+Connection ~ 9700 6050
+Wire Wire Line
+	9700 6050 9900 6050
+Wire Wire Line
+	9150 6050 8650 6050
+Wire Wire Line
+	8250 6050 8250 5900
+Connection ~ 9150 6050
+Wire Wire Line
+	8450 6050 8450 5900
+Connection ~ 8450 6050
+Wire Wire Line
+	8450 6050 8250 6050
+Wire Wire Line
+	8650 6050 8650 5900
+Connection ~ 8650 6050
+Wire Wire Line
+	8650 6050 8450 6050
+Wire Wire Line
+	8450 4950 9150 4950
+Wire Wire Line
+	9150 4850 9150 4950
+Connection ~ 9150 4950
+Wire Wire Line
+	9150 4950 9900 4950
 $EndSCHEMATC

Commit message: updated revb
Parts:
- removed D2, D3: LED_RGBA, LED_THT:LED_D5.0mm-4_RGB_Wide_Pins, symbol Device:LED_RGBA
- removed J1, J2, J6: Conn_01x02, Connector_PinHeader_2.54mm:PinHeader_1x02_P2.54mm_Vertical, symbol Connector_Generic:Conn_01x02
- removed J4: Conn_01x03, Connector_PinHeader_2.54mm:PinHeader_1x03_P2.54mm_Vertical, symbol Connector_Generic:Conn_01x03
- removed R4, R5, R7, R8: R, Resistor_SMD:R_0805_2012Metric_Pad1.15x1.40mm_HandSolder, symbol Device:R
- added D2, D3: LED, LED_SMD:LED_1206_3216Metric_Pad1.42x1.75mm_HandSolder, symbol Device:LED
- added J1, J6: AudioJack2, Connector_PinHeader_2.54mm:PinHeader_1x02_P2.54mm_Vertical, symbol Connector:AudioJack2
- added J2: Barrel_Jack, Connector_PinHeader_2.54mm:PinHeader_1x02_P2.54mm_Vertical, symbol Connector:Barrel_Jack
- added RV1: B10K, Connector_PinHeader_2.54mm:PinHeader_1x03_P2.54mm_Vertical, symbol Device:R_POT
- R6, R9: value R -> 1K
Connections:
- wire segments 77 -> 61
Other:
- moved on the sheet: C1, C2, C7, C9, R1, R2, R3, R6, R9, U2
