File: OverdrivePedal_RevB/PosNeg5V_PSU.sch (KiCad schematic (older format))
At the start: 9 parts, among them U2 NCP1729, U3 MIC5233-5.0YM5-TR, U4 MIC5270-5.0YM5-TR

Commit message: modified RevB
Parts:
- removed C4, C5: 10uF, Capacitor_SMD:CP_Elec_4x5.7, symbol Device:CP
- removed U2: NCP1729, Package_TO_SOT_SMD:SOT-23-6_Handsoldering, symbol NCP1729:NCP1729
- removed U3: MIC5233-5.0YM5-TR, Package_TO_SOT_SMD:SOT-23-5_HandSoldering, symbol MIC5233:MIC5233YM5
- removed U4: MIC5270-5.0YM5-TR, Package_TO_SOT_SMD:SOT-23-5_HandSoldering, symbol MIC5270YM5:MIC5270YM5
- added C10: 330nF, Capacitor_SMD:C_0805_2012Metric_Pad1.15x1.40mm_HandSolder, symbol Device:C
- added C11, C4, C5: 1uF, Capacitor_SMD:C_0805_2012Metric_Pad1.15x1.40mm_HandSolder, symbol Device:C
- added U3: TPS60400, Package_TO_SOT_SMD:SOT-23-5_HandSoldering, symbol TPS6040x:TPS60400
- added U4: KIA78L05T, Package_TO_SOT_SMD:SOT-89-3, symbol Regulator_Linear:MC78L05_SOT89
- added U5: XC6902N501PR-G, Package_TO_SOT_SMD:SOT-89-3, symbol Regulator_Linear:L79L05_SOT89
- C3: value 100nF -> 1uF
- C8: value 2.2uF -> 100nF
- D1: value D_Schottky -> BYS12-90
Connections:
- wire segments 39 -> 38
- no-connect marks 3 -> 0
Other:
- note added: "LDO Min VIn: -16V"
- note added: "Max Vin: 30V"
- moved on the sheet: C3

Commit message: updated revb
Parts:
- removed C11, C6: 1uF, Capacitor_SMD:C_0805_2012Metric_Pad1.15x1.40mm_HandSolder, symbol Device:C
- removed U5: XC6902N501PR-G, Package_TO_SOT_SMD:SOT-89-3, symbol Regulator_Linear:L79L05_SOT89
- D1: footprint Diode_SMD:D_SMA_Handsoldering -> Diode_SMD:D_SOD-123F
Connections:
- net labels removed: -5V_REG
- wire segments 38 -> 27
Other:
- note removed: "LDO Min VIn: -16V"
- moved on the sheet: C3, C4, C5, U3
Changed lines of the file:
@@
 L power:GNDS #PWR011
 U 1 1 5E625BFF
-P 3050 5225
+P 6750 5225
 AR Path="/5E6165F4/5E625BFF" Ref="#PWR011"  Part="1"
 AR Path="/5E6A8284/5E625BFF" Ref="#PWR?"  Part="1"
-F 0 "#PWR011" H 3050 4975 50  0001 C CNN
-F 1 "GNDS" H 3055 5052 50  0000 C CNN
-F 2 "" H 3050 5225 50  0001 C CNN
-F 3 "" H 3050 5225 50  0001 C CNN
-	1    3050 5225
-	1    0    0    -1
-$EndComp
-$Comp
-L power:GNDS #PWR?
-U 1 1 5E62DA80
-P 6250 5450
-AR Path="/5E62DA80" Ref="#PWR?"  Part="1"
-AR Path="/5E6165F4/5E62DA80" Ref="#PWR015"  Part="1"
-AR Path="/5E6A8284/5E62DA80" Ref="#PWR?"  Part="1"
-F 0 "#PWR015" H 6250 5200 50  0001 C CNN
-F 1 "GNDS" H 6255 5277 50  0000 C CNN
-F 2 "" H 6250 5450 50  0001 C CNN
-F 3 "" H 6250 5450 50  0001 C CNN
-	1    6250 5450
-	1    0    0    -1
-$EndComp
-Connection ~ 6250 5350
-Wire Wire Line
-	6250 5350 6250 5450
-Wire Wire Line
-	7700 4600 7700 4250
-Wire Wire Line
-	7700 4900 7700 5350
-Connection ~ 7700 4250
-Text Label 8200 4250 2    50   ~ 0
--5V_REG
+F 0 "#PWR011" H 6750 4975 50  0001 C CNN
+F 1 "GNDS" H 6755 5052 50  0000 C CNN
+F 2 "" H 6750 5225 50  0001 C CNN
+F 3 "" H 6750 5225 50  0001 C CNN
+	1    6750 5225
+	1    0    0    -1
+$EndComp
 Text HLabel 1350 1900 0    50   Input ~ 0
 +9V_IN
@@
 Text HLabel 10150 4250 2    50   Input ~ 0
 -5V
-Wire Wire Line
-	6250 4550 6250 5350
 $Comp
 L Device:D_Schottky D1
@@
 F 0 "D1" H 2600 1684 50  0000 C CNN
 F 1 "BYS12-90" H 2600 1775 50  0000 C CNN
-F 2 "Diode_SMD:D_SMA_Handsoldering" H 2600 1900 50  0001 C CNN
+F 2 "Diode_SMD:D_SOD-123F" H 2600 1900 50  0001 C CNN
 F 3 "~" H 2600 1900 50  0001 C CNN
 	1    2600 1900
@@
 Wire Wire Line
 	6400 1900 7700 1900
-Wire Wire Line
-	6250 5350 7700 5350
-Wire Wire Line
-	6550 4250 7700 4250
 $Comp
 L Device:C C8
@@
 $EndComp
 $Comp
-L Device:C C6
-U 1 1 5E68B0FD
-P 7700 4750
-AR Path="/5E6165F4/5E68B0FD" Ref="C6"  Part="1"
-AR Path="/5E6A8284/5E68B0FD" Ref="C?"  Part="1"
-F 0 "C6" H 7815 4796 50  0000 L CNN
-F 1 "1uF" H 7815 4705 50  0000 L CNN
-F 2 "Capacitor_SMD:C_0805_2012Metric_Pad1.15x1.40mm_HandSolder" H 7738 4600 50  0001 C CNN
-F 3 "~" H 7700 4750 50  0001 C CNN
-	1    7700 4750
-	1    0    0    -1
-$EndComp
-$Comp
 L Device:C C3
 U 1 1 5E6ACD77
-P 1650 4550
+P 5350 4550
 AR Path="/5E6165F4/5E6ACD77" Ref="C3"  Part="1"
 AR Path="/5E6A8284/5E6ACD77" Ref="C?"  Part="1"
-F 0 "C3" H 1765 4596 50  0000 L CNN
-F 1 "1uF" H 1765 4505 50  0000 L CNN
-F 2 "Capacitor_SMD:C_0805_2012Metric_Pad1.15x1.40mm_HandSolder" H 1688 4400 50  0001 C CNN
-F 3 "~" H 1650 4550 50  0001 C CNN
-	1    1650 4550
-	1    0    0    -1
-$EndComp
-Text Label 750  4250 0    50   ~ 0
+F 0 "C3" H 5465 4596 50  0000 L CNN
+F 1 "1uF" H 5465 4505 50  0000 L CNN
+F 2 "Capacitor_SMD:C_0805_2012Metric_Pad1.15x1.40mm_HandSolder" H 5388 4400 50  0001 C CNN
+F 3 "~" H 5350 4550 50  0001 C CNN
+	1    5350 4550
+	1    0    0    -1
+$EndComp
+Text Label 4450 4250 0    50   ~ 0
 +5V_REG
-Text Label 4550 4250 2    50   ~ 0
+Text Label 8675 4250 2    50   ~ 0
 -5V_POL
 $Comp
@@
 Wire Wire Line
 	4925 3300 6100 3300
-$Comp
-L Regulator_Linear:L79L05_SOT89 U5
-U 1 1 5E690159
-P 6250 4250
-F 0 "U5" H 6250 3900 50  0000 C CNN
-F 1 "XC6902N501PR-G " H 6250 3975 50  0000 C CNN
-F 2 "Package_TO_SOT_SMD:SOT-89-3" H 6250 4050 50  0001 C CIN
-F 3 "https://datasheet.lcsc.com/szlcsc/1810010340_Torex-Semicon-XC6902N501PR-G_C165898.pdf" H 6250 4250 50  0001 C CNN
-	1    6250 4250
-	1    0    0    1
-$EndComp
 Text Notes 5850 1775 0    50   ~ 0
 Max Vin: 30V
@@
 L TPS6040x:TPS60400 U3
 U 1 1 5E6AE9A9
-P 2400 4500
-F 0 "U3" H 2400 5105 50  0000 C CNN
-F 1 "TPS60400" H 2400 5014 50  0000 C CNN
-F 2 "Package_TO_SOT_SMD:SOT-23-5_HandSoldering" H 2400 4923 50  0000 C CNN
-F 3 "http://www.ti.com/lit/ds/symlink/tps60402.pdf" H 2350 4650 50  0001 C CNN
-	1    2400 4500
-	1    0    0    -1
-$EndComp
-Wire Wire Line
-	2800 4250 3500 4250
-Wire Wire Line
-	750  4250 1250 4250
-Wire Wire Line
-	3050 4750 3050 5225
-Wire Wire Line
-	3050 4750 2800 4750
-Wire Wire Line
-	1650 4400 1650 4350
-Wire Wire Line
-	1650 4350 2000 4350
-Wire Wire Line
-	2000 4750 1650 4750
-Wire Wire Line
-	1650 4750 1650 4700
+P 6100 4500
+AR Path="/5E6AE9A9" Ref="U3"  Part="1"
+AR Path="/5E6165F4/5E6AE9A9" Ref="U3"  Part="1"
+F 0 "U3" H 6100 5105 50  0000 C CNN
+F 1 "TPS60400" H 6100 5014 50  0000 C CNN
+F 2 "Package_TO_SOT_SMD:SOT-23-5_HandSoldering" H 6100 4923 50  0000 C CNN
+F 3 "http://www.ti.com/lit/ds/symlink/tps60402.pdf" H 6050 4650 50  0001 C CNN
+	1    6100 4500
+	1    0    0    -1
+$EndComp
+Wire Wire Line
+	6500 4250 7200 4250
+Wire Wire Line
+	4450 4250 4950 4250
+Wire Wire Line
+	6750 4750 6750 5225
+Wire Wire Line
+	6750 4750 6500 4750
+Wire Wire Line
+	5350 4400 5350 4350
+Wire Wire Line
+	5350 4350 5700 4350
+Wire Wire Line
+	5700 4750 5350 4750
+Wire Wire Line
+	5350 4750 5350 4700
 $Comp
 L Device:C C4
 U 1 1 5E6B5D25
-P 1250 4550
+P 4950 4550
 AR Path="/5E6165F4/5E6B5D25" Ref="C4"  Part="1"
 AR Path="/5E6A8284/5E6B5D25" Ref="C?"  Part="1"
-F 0 "C4" H 1365 4596 50  0000 L CNN
-F 1 "1uF" H 1365 4505 50  0000 L CNN
-F 2 "Capacitor_SMD:C_0805_2012Metric_Pad1.15x1.40mm_HandSolder" H 1288 4400 50  0001 C CNN
-F 3 "~" H 1250 4550 50  0001 C CNN
-	1    1250 4550
-	1    0    0    -1
-$EndComp
-Wire Wire Line
-	1250 4400 1250 4250
-Connection ~ 1250 4250
-Wire Wire Line
-	1250 4250 2000 4250
+F 0 "C4" H 5065 4596 50  0000 L CNN
+F 1 "1uF" H 5065 4505 50  0000 L CNN
+F 2 "Capacitor_SMD:C_0805_2012Metric_Pad1.15x1.40mm_HandSolder" H 4988 4400 50  0001 C CNN
+F 3 "~" H 4950 4550 50  0001 C CNN
+	1    4950 4550
+	1    0    0    -1
+$EndComp
+Wire Wire Line
+	4950 4400 4950 4250
+Connection ~ 4950 4250
+Wire Wire Line
+	4950 4250 5700 4250
 $Comp
 L power:GNDS #PWR0106
 U 1 1 5E6B6E92
-P 1250 5175
+P 4950 5175
 AR Path="/5E6165F4/5E6B6E92" Ref="#PWR0106"  Part="1"
 AR Path="/5E6A8284/5E6B6E92" Ref="#PWR?"  Part="1"
-F 0 "#PWR0106" H 1250 4925 50  0001 C CNN
-F 1 "GNDS" H 1255 5002 50  0000 C CNN
-F 2 "" H 1250 5175 50  0001 C CNN
-F 3 "" H 1250 5175 50  0001 C CNN
-	1    1250 5175
-	1    0    0    -1
-$EndComp
-Wire Wire Line
-	1250 4700 1250 5175
+F 0 "#PWR0106" H 4950 4925 50  0001 C CNN
+F 1 "GNDS" H 4955 5002 50  0000 C CNN
+F 2 "" H 4950 5175 50  0001 C CNN
+F 3 "" H 4950 5175 50  0001 C CNN
+	1    4950 5175
+	1    0    0    -1
+$EndComp
+Wire Wire Line
+	4950 4700 4950 5175
 $Comp
 L Device:C C5
 U 1 1 5E6B7FA9
-P 3500 4550
+P 7200 4550
 AR Path="/5E6165F4/5E6B7FA9" Ref="C5"  Part="1"
 AR Path="/5E6A8284/5E6B7FA9" Ref="C?"  Part="1"
-F 0 "C5" H 3615 4596 50  0000 L CNN
-F 1 "1uF" H 3615 4505 50  0000 L CNN
-F 2 "Capacitor_SMD:C_0805_2012Metric_Pad1.15x1.40mm_HandSolder" H 3538 4400 50  0001 C CNN
-F 3 "~" H 3500 4550 50  0001 C CNN
-	1    3500 4550
-	1    0    0    -1
-$EndComp
-Wire Wire Line
-	3500 4400 3500 4250
+F 0 "C5" H 7315 4596 50  0000 L CNN
+F 1 "1uF" H 7315 4505 50  0000 L CNN
+F 2 "Capacitor_SMD:C_0805_2012Metric_Pad1.15x1.40mm_HandSolder" H 7238 4400 50  0001 C CNN
+F 3 "~" H 7200 4550 50  0001 C CNN
+	1    7200 4550
+	1    0    0    -1
+$EndComp
+Wire Wire Line
+	7200 4400 7200 4250
 $Comp
 L power:GNDS #PWR0107
 U 1 1 5E6B7FB0
-P 3500 5175
+P 7200 5175
 AR Path="/5E6165F4/5E6B7FB0" Ref="#PWR0107"  Part="1"
 AR Path="/5E6A8284/5E6B7FB0" Ref="#PWR?"  Part="1"
-F 0 "#PWR0107" H 3500 4925 50  0001 C CNN
-F 1 "GNDS" H 3505 5002 50  0000 C CNN
-F 2 "" H 3500 5175 50  0001 C CNN
-F 3 "" H 3500 5175 50  0001 C CNN
-	1    3500 5175
-	1    0    0    -1
-$EndComp
-Wire Wire Line
-	3500 4700 3500 5175
-Connection ~ 3500 4250
-Wire Wire Line
-	3500 4250 5350 4250
-$Comp
-L Device:C C11
-U 1 1 5E6BD31D
-P 5350 4750
-AR Path="/5E6165F4/5E6BD31D" Ref="C11"  Part="1"
-AR Path="/5E6A8284/5E6BD31D" Ref="C?"  Part="1"
-F 0 "C11" H 5465 4796 50  0000 L CNN
-F 1 "1uF" H 5465 4705 50  0000 L CNN
-F 2 "Capacitor_SMD:C_0805_2012Metric_Pad1.15x1.40mm_HandSolder" H 5388 4600 50  0001 C CNN
-F 3 "~" H 5350 4750 50  0001 C CNN
-	1    5350 4750
-	1    0    0    -1
-$EndComp
-Wire Wire Line
-	5350 4600 5350 4250
-Connection ~ 5350 4250
-Wire Wire Line
-	5350 4250 5950 4250
-Wire Wire Line
-	5350 4900 5350 5350
-Wire Wire Line
-	5350 5350 6250 5350
-Text Notes 5850 4100 0    50   ~ 0
-LDO Min VIn: -16V
+F 0 "#PWR0107" H 7200 4925 50  0001 C CNN
+F 1 "GNDS" H 7205 5002 50  0000 C CNN
+F 2 "" H 7200 5175 50  0001 C CNN
+F 3 "" H 7200 5175 50  0001 C CNN
+	1    7200 5175
+	1    0    0    -1
+$EndComp
+Wire Wire Line
+	7200 4700 7200 5175
 Wire Wire Line
 	7700 1900 10200 1900
-Wire Wire Line
-	7700 4250 10150 4250
 $Comp
 L power:PWR_FLAG #FLG0102
@@
 	1    0    0    -1
 $EndComp
+Wire Wire Line
+	7200 4250 10150 4250
+Connection ~ 7200 4250
 $EndSCHEMATC

Commit message: updated revb design
- Added solidstate ICs for bypass switching to allow for mom. footswitch
- Added STM32L011 MCU
-  Added SE82XX (SOT23) LDOs for 5V and 3V3 rails
Parts:
- removed U4: KIA78L05T, Package_TO_SOT_SMD:SOT-89-3, symbol Regulator_Linear:MC78L05_SOT89
- added C11, C12: 10uF, Capacitor_SMD:C_0805_2012Metric_Pad1.15x1.40mm_HandSolder, symbol Device:C
- added U7: SE8233X2, Package_TO_SOT_SMD:SOT-23, symbol Regulator_Linear:MCP1700-5002E_SOT23
- added U8: SE8250X2, Package_TO_SOT_SMD:SOT-23, symbol Regulator_Linear:MCP1700-5002E_SOT23
- C10: value 330nF -> 1uF
- C8: value 100nF -> 1uF
Connections:
- net labels added: +3V3_REG, 3V3
- wire segments 27 -> 42
Other:
- note removed: "Max Vin: 30V"
- moved on the sheet: C3, C4, C5, D1, U3
